Commit message: Camera working in simulation - publishes on /camera/image_raw

File: urdf/soft_wrist.urdf.xacro (robot description, xacro)
@@ -92,3 +92,41 @@
     </plugin>
   </gazebo>
+  <!-- Simulated camera attached to soft wrist — mirrors real Pi Camera -->
+  <link name="camera_link">
+    <visual>
+      <geometry>
+        <box size="0.025 0.024 0.009"/>
+      </geometry>
+      <material name="teal"/>
+    </visual>
+    <inertial>
+      <mass value="0.03"/>
+      <inertia ixx="0.00001" ixy="0" ixz="0" iyy="0.00001" iyz="0" izz="0.00001"/>
+    </inertial>
+  </link>
+  <joint name="wrist_to_camera" type="fixed">
+    <parent link="soft_wrist_assembly"/>
+    <child link="camera_link"/>
+    <origin xyz="0.03 0 -0.05" rpy="0 1.5708 0"/>
+  </joint>
+  <gazebo reference="camera_link">
+    <sensor name="camera" type="camera">
+      <camera>
+        <horizontal_fov>1.047</horizontal_fov>
+        <image>
+          <width>640</width>
+          <height>480</height>
+          <format>R8G8B8</format>
+        </image>
+        <clip>
+          <near>0.01</near>
+          <far>5.0</far>
+        </clip>
+      </camera>
+      <always_on>1</always_on>
+      <update_rate>10</update_rate>
+      <visualize>true</visualize>
+      <topic>/camera/image_raw</topic>
+    </sensor>
+  </gazebo>
 </robot>

Commit message: Add ArUco detection node, overhead camera, Z compliance pipeline working

File: urdf/soft_wrist.urdf.xacro (robot description, xacro)
@@ -108,5 +108,5 @@
     <parent link="soft_wrist_assembly"/>
     <child link="camera_link"/>
-    <origin xyz="0.03 0 -0.05" rpy="0 1.5708 0"/>
+    <origin xyz="0 0 -0.15" rpy="0 0 0"/>
   </joint>
   <gazebo reference="camera_link">
