Commit message: Fix soft wrist mesh attachment to UR5e tool0 - calibrated via Gazebo drag-and-drop, CB1-3 joints restored, camera restored

File: urdf/soft_wrist.urdf.xacro (robot description, xacro)
@@ -6,4 +6,5 @@
   <xacro:arg name="tf_prefix"         default=""/>
   <xacro:include filename="$(find ur_description)/urdf/ur_macro.xacro"/>
+  <xacro:include filename="$(find soft_wrist_sim)/urdf/soft_wrist_mechanism.urdf.xacro"/>
   <link name="world"/>
   <xacro:ur_robot
@@ -27,28 +28,12 @@
     <color rgba="0.18 0.80 0.71 1.0"/>
   </material>
-  <link name="soft_wrist_assembly">
-    <visual>
-      <geometry>
-        <mesh filename="package://soft_wrist_sim/meshes/assembly.stl" scale="1 1 1"/>
-      </geometry>
-      <material name="teal"/>
-    </visual>
-    <collision>
-      <geometry>
-        <box size="0.06 0.06 0.11"/>
-      </geometry>
-    </collision>
-    <inertial>
-      <mass value="0.3"/>
-      <inertia ixx="0.0001" ixy="0" ixz="0"
-               iyy="0.0001" iyz="0"
-               izz="0.0001"/>
-    </inertial>
-  </link>
-  <joint name="flange_to_wrist" type="fixed">
-    <parent link="tool0"/>
-    <child link="soft_wrist_assembly"/>
-    <origin xyz="-0.045 -0.023 0.02" rpy="0 0 0"/>
-  </joint>
+  <material name="light_blue">
+    <color rgba="0.529 0.808 0.922 1.0"/>
+  </material>
+  <!-- Soft wrist parallel mechanism attached to UR5e tool0 -->
+  <xacro:soft_wrist_mechanism prefix="" parent="tool0">
+    <origin xyz="-0.0164 0.0166 0.0098" rpy="2.9887 0 -1.5708"/>
+  </xacro:soft_wrist_mechanism>
+  <!-- ros2_control — UR5e arm + 3 soft wrist servos -->
   <ros2_control name="GazeboSimSystem" type="system">
     <hardware>
@@ -85,4 +70,32 @@
       <state_interface name="velocity"/>
     </joint>
+    Soft wrist Dynamixel servo joints (commented below)
+    <joint name="CB1">
+      <command_interface name="position">
+        <param name="min">-0.785</param>
+        <param name="max">0.785</param>
+      </command_interface>
+      <state_interface name="position"><param name="initial_value">0.0</param></state_interface>
+      <state_interface name="velocity"/>
+      <state_interface name="effort"/>
+    </joint>
+    <joint name="CB2">
+      <command_interface name="position">
+        <param name="min">-0.785</param>
+        <param name="max">0.785</param>
+      </command_interface>
+      <state_interface name="position"><param name="initial_value">0.0</param></state_interface>
+      <state_interface name="velocity"/>
+      <state_interface name="effort"/>
+    </joint>
+    <joint name="CB3">
+      <command_interface name="position">
+        <param name="min">-0.785</param>
+        <param name="max">0.785</param>
+      </command_interface>
+      <state_interface name="position"><param name="initial_value">0.0</param></state_interface>
+      <state_interface name="velocity"/>
+      <state_interface name="effort"/>
+    </joint>
   </ros2_control>
   <gazebo>
@@ -92,5 +105,5 @@
     </plugin>
   </gazebo>
-  <!-- Simulated camera attached to soft wrist — mirrors real Pi Camera -->
+  Camera mounted on sw_base looking down
   <link name="camera_link">
     <visual>
@@ -102,11 +115,13 @@
     <inertial>
       <mass value="0.03"/>
-      <inertia ixx="0.00001" ixy="0" ixz="0" iyy="0.00001" iyz="0" izz="0.00001"/>
+      <inertia ixx="0.00001" ixy="0" ixz="0"
+               iyy="0.00001" iyz="0"
+               izz="0.00001"/>
     </inertial>
   </link>
   <joint name="wrist_to_camera" type="fixed">
-    <parent link="soft_wrist_assembly"/>
+    <parent link="sw_base"/>
     <child link="camera_link"/>
-    <origin xyz="0 0 -0.15" rpy="0 0 0"/>
+    <origin xyz="0 0 0.02" rpy="0 3.1416 0"/>
   </joint>
   <gazebo reference="camera_link">

Commit message: Add admittance control pipeline: wrench estimator, single and 3-DOF admittance controllers, live plotting. Fix TF publishing (ignore_timestamp), calibrate mesh attachment to tool0, fix collision geometry, add camera pose to world file.

File: urdf/soft_wrist.urdf.xacro (robot description, xacro)
@@ -79,4 +79,5 @@
       <state_interface name="velocity"/>
       <state_interface name="effort"/>
+      <param name="position_proportional_gain">20.0</param>
     </joint>
     <joint name="CB2">
@@ -88,4 +89,5 @@
       <state_interface name="velocity"/>
       <state_interface name="effort"/>
+      <param name="position_proportional_gain">20.0</param>
     </joint>
     <joint name="CB3">
@@ -97,4 +99,5 @@
       <state_interface name="velocity"/>
       <state_interface name="effort"/>
+      <param name="position_proportional_gain">20.0</param>
     </joint>
   </ros2_control>

File: urdf/soft_wrist_mechanism.urdf.xacro (robot description, xacro)
@@ -7,4 +7,14 @@
       <child link="${prefix}sw_base"/>
     </joint>
+    <gazebo reference="${prefix}tool0_to_soft_wrist_base">
+      <sensor name="${prefix}wrist_ft_sensor" type="force_torque">
+        <always_on>true</always_on>
+        <update_rate>100</update_rate>
+        <force_torque>
+          <frame>child</frame>
+          <measure_direction>child_to_parent</measure_direction>
+        </force_torque>
+      </sensor>
+    </gazebo>
     <!-- Full mechanism as single merged mesh — no splitting ever -->
     <link name="${prefix}sw_base">
@@ -23,7 +33,7 @@
         </material>
       </visual>
-      <collision>
-        <origin xyz="0 0 0" rpy="0 0 0"/>
-        <geometry><box size="0.08 0.08 0.08"/></geometry>
+      <collision name="${prefix}sw_base_collision">
+        <origin xyz="0.022 -0.0245 -0.0595" rpy="0 0 0"/>
+        <geometry><box size="0.142 0.127 0.175"/></geometry>
       </collision>
     </link>
@@ -36,5 +46,5 @@
       <axis xyz="0 0 -1"/>
       <limit lower="-0.785" upper="0.785" effort="1.8" velocity="3.14"/>
-      <dynamics damping="100.0" friction="10.0"/>
+      <dynamics damping="0.5" friction="0.1"/>
     </joint>
     <link name="${prefix}sw_CB1">
@@ -52,5 +62,5 @@
       <axis xyz="0 0 -1"/>
       <limit lower="-0.785" upper="0.785" effort="1.8" velocity="3.14"/>
-      <dynamics damping="100.0" friction="10.0"/>
+      <dynamics damping="0.5" friction="0.1"/>
     </joint>
     <link name="${prefix}sw_CB2">
@@ -69,5 +79,5 @@
       <axis xyz="0 0 -1"/>
       <limit lower="-0.785" upper="0.785" effort="1.8" velocity="3.14"/>
-      <dynamics damping="100.0" friction="10.0"/>
+      <dynamics damping="0.5" friction="0.1"/>
     </joint>
     <link name="${prefix}sw_CB3">
